File: board/woodBLDCdeveloper/woodBLDCdeveloper.kicad_sch (KiCad schematic)
At the start: 78 parts, among them J1 Conn_01x04, J2 Conn_01x06, J3 Conn_01x01, J4 Conn_01x01, J5 Conn_01x04, J6 Conn_01x01, J7 Conn_01x01, J8 Conn_01x01, Q1 Q_NMOS_GDS, Q2 Q_NMOS_GDS, Q3 Q_NMOS_GDS, Q4 Q_NMOS_GDS, Q5 Q_NMOS_GDS, Q6 Q_NMOS_GDS, U1 SCM3728ASA, U2 SCM3728ASA, U3 Si8641BA-B-IU, U4 K78U03-500R3, U5 MCP1792x-3302xCB, U6 PICkit3, U7 dsPIC33CH64MP202T, U8 DRV8328BRUY, U9 Opamp_Quad, Y1 16MHz

Commit message: 回路設計と部品割り当て終わった
Parts:
- removed U5: MCP1792x-3302xCB, Package_TO_SOT_SMD:SOT-23, symbol Regulator_Linear:MCP1792x-3302xCB
- added U5: NCV8163ASN330T1G, Package_SO:TSOP-5_1.65x3.05mm_P0.95mm, symbol 0_kicad_wood:NCV8163ASN330T1G
- C1, C13, C14, C15, C17, C18, C2, C20, C21, C22, C23, C3, C4, C5, C6: footprint (none) -> Capacitor_SMD:C_0603_1608Metric_Pad1.08x0.95mm_HandSolder
- C10: renamed from C11; footprint (none) -> Capacitor_SMD:C_0805_2012Metric_Pad1.18x1.45mm_HandSolder
- C11: renamed from C9; value 2.2u/100V -> 1u; footprint (none) -> Capacitor_SMD:C_0603_1608Metric_Pad1.08x0.95mm_HandSolder
- C12: value 2.2u -> 1u; footprint (none) -> Capacitor_SMD:C_0603_1608Metric_Pad1.08x0.95mm_HandSolder
- C16: value 10u/100V -> 47u/100V; footprint (none) -> Capacitor_THT:CP_Radial_D10.0mm_P5.00mm
- C19: footprint (none) -> Capacitor_SMD:C_0805_2012Metric_Pad1.18x1.45mm_HandSolder
- C7: footprint (none) -> Capacitor_THT:CP_Radial_D12.5mm_P5.00mm
- C8: footprint (none) -> Capacitor_SMD:C_1210_3225Metric_Pad1.33x2.70mm_HandSolder
- C9: renamed from C10; footprint (none) -> Capacitor_SMD:C_1210_3225Metric_Pad1.33x2.70mm_HandSolder
- D1, D2, D3, D4: footprint (none) -> LED_SMD:LED_0603_1608Metric_Pad1.05x0.95mm_HandSolder
- J1: footprint (none) -> Connector_JST:JST_XH_S4B-XH-A_1x04_P2.50mm_Horizontal
- J2: footprint (none) -> Connector_JST:JST_XH_S6B-XH-A_1x06_P2.50mm_Horizontal
- J3, J4, J6, J7, J8: footprint (none) -> MountingHole:MountingHole_2.2mm_M2_Pad_Via
- J5: footprint (none) -> Connector_JST:JST_XH_B4B-XH-A_1x04_P2.50mm_Vertical
- Q1, Q2, Q3, Q4, Q5, Q6: footprint (none) -> Package_TO_SOT_SMD:TO-252-2
- R1, R10, R11, R12, R13, R14, R15, R18, R19, R2, R20, R21, R22, R23, R24, R25, R26, R27, R3, R4, R5, R6, R7, R8, R9: footprint (none) -> Resistor_SMD:R_0603_1608Metric_Pad0.98x0.95mm_HandSolder
- R16, R17: footprint (none) -> Resistor_SMD:R_1206_3216Metric_Pad1.30x1.75mm_HandSolder
- U1, U2: footprint (none) -> Package_SO:SOIC-8_3.9x4.9mm_P1.27mm
- U4: value K78U03-500R3 -> K78U05-500R3; footprint (none) -> 0_kicad_wood:K78Uxx-500R3
- U6: footprint (none) -> Connector_PinHeader_2.54mm:PinHeader_1x06_P2.54mm_Horizontal
- U7: footprint (none) -> Package_SO:SSOP-28_5.3x10.2mm_P0.65mm
- U8: footprint (none) -> Package_DFN_QFN:QFN-28-1EP_4x4mm_P0.4mm_EP2.6x2.6mm
- U9: footprint (none) -> Package_SO:TSSOP-14_4.4x5mm_P0.65mm
- Y1: footprint (none) -> Crystal:Resonator_SMD_Murata_CSTxExxV-3Pin_3.0x1.1mm
Connections:
- net +3.3VA is gone; now on net +3.3VP: C12.1, C15.1, C23.1, R24.2, U7.5 (AVDD), U9.4 (V+)
- net +3.3VP: now also U5.5 (OUT); no longer C10.1, U4.3 (VOUT)
- net +BATT: no longer C11.1
- net GNDPWR: now also U5.2 (GND)
- new net: C10.1, C11.1, U4.3 (VOUT), U5.1 (IN), U5.3 (EN)
- no-connect marks 6 -> 7
Other:
- moved on the sheet: C10, C11, C12, C7, C8, C9, D1, J3, J4, R1, U4
